File: Alexandria-ng/Alexandria-ng.kicad_sch (KiCad schematic)
At the start: 29 parts, among them J13 +3.3V, SW1 RST, U1 RTL8367S-CG, Y1 25M

Commit message: sch: Add mounting holes
Parts:
- added H1, H2, H3, H4: M2.5, MountingHole:MountingHole_2.7mm_M2.5_ISO7380_Pad, symbol Mechanical:MountingHole_Pad
Connections:
- net GND: now also H1.1, H2.1, H3.1, H4.1
Other:
- note added: "For MangoPi"
