File: Alexandria-ng/Alexandria-ng.kicad_pcb (KiCad board)
At the start: 4 copper layers, 150 x 105 mm, 87 parts, among them J1 Eth0, J10 PoE3, J11 PoE4, J12 FFC, J13 +3.3V, J14 I²C, J2 Eth1, J3 Eth2, J4 Eth3, J5 Eth4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

Commit message: Back silkscreen
Parts:
- moved D1 33.1 mm to (186.5, 116.3)
- moved R4 33.1 mm to (190.0, 116.3)
Routing:
- net +3.3V: track 190.5 -> 186.8 mm
Other:
- board text added: "LibrEther - Project Alexandria 5-port switch with RGMII/HSGMII Version 2.00 drawn 2023-06-20 by CsokiCraft https://bence98.github.io/LibreEther"

Commit message: More silkscreen work
Parts:
- moved D1 5.52 mm to (190.6, 112.6)
- moved R4 5.52 mm to (194.1, 112.6)
Routing:
- net +3.3V: track 186.8 -> 192.5 mm

Commit message: Re-fill zones, fix some DRC warnings
Routing:
- net GND: vias 208 -> 209
Other:
- board size 150 x 105 mm -> 150.2 x 105 mm
